Commit message: Added dummy controllers for passive joints

File: project_one/urdf/toy_car.urdf.xacro (robot description, xacro)
@@ -1055,4 +1055,25 @@
       <state_interface name="velocity"/>
     </joint>
+    <!-- Dummy Controller for Passive Joints -->
+    <joint name="front_left_axle_joint">
+      <state_interface name="position"/>
+      <state_interface name="velocity"/>
+    </joint>
+    <joint name="front_right_axle_joint">
+      <state_interface name="position"/>
+      <state_interface name="velocity"/>
+    </joint>
+    <joint name="trailer_joint">
+      <state_interface name="position"/>
+      <state_interface name="velocity"/>
+    </joint>
+    <joint name="trailer_left_axle_joint">
+      <state_interface name="position"/>
+      <state_interface name="velocity"/>
+    </joint>
+    <joint name="trailer_right_axle_joint">
+      <state_interface name="position"/>
+      <state_interface name="velocity"/>
+    </joint>
   </ros2_control>
   <gazebo>
