Commit message: Updated Robot Model and Kinematics

File: project_two/urdf/robot_arm.urdf.xacro (robot description, xacro)
@@ -1,5 +1,9 @@
 <?xml version="1.0" ?>
+<!-- This URDF was automatically created by SolidWorks to URDF Exporter! Originally created by Stephen Brawner (brawner@gmail.com)
+     Commit Version: 1.6.0-4-g7f85cfe  Build Version: 1.6.7995.38578
+     For more information, please see http://wiki.ros.org/sw_urdf_exporter -->
 <robot
   name="robot_arm" xmlns:xacro="http://ros.org/wiki/xacro">
+  <!-- Gazebo Color Plugins -->
   <xacro:macro name="body_color">
     <visual>
@@ -22,4 +26,25 @@
     </visual>
   </xacro:macro>
+  <xacro:macro name="base_color">
+    <visual>
+      <material>
+        <ambient>0.41569 0.67451 1 1</ambient>
+        <diffuse>0.41569 0.67451 1 1</diffuse>
+        <specular>0.1 0.1 0.1 1</specular>
+        <emissive>0 0 0 0</emissive>
+      </material>
+    </visual>
+  </xacro:macro>
+  <xacro:macro name="tool_color">
+    <visual>
+      <material>
+        <ambient>0.19608 0.19608 0.19608 1</ambient>
+        <diffuse>0.19608 0.19608 0.19608 1</diffuse>
+        <specular>0.1 0.1 0.1 1</specular>
+        <emissive>0 0 0 0</emissive>
+      </material>
+    </visual>
+  </xacro:macro>
+  <!-- World Link for Fixed Base -->
   <link name="world" />
   <link
@@ -27,15 +52,15 @@
     <inertial>
       <origin
-        xyz="0.000818930716522579 -0.000818930139439305 0.0140278111957652"
-        rpy="0 0 0" />
-      <mass
-        value="0.365058052116186" />
-      <inertia
-        ixx="0.00051380644225505"
-        ixy="-1.25381433478329E-05"
-        ixz="3.47062873674803E-08"
-        iyy="0.000513806425545493"
-        iyz="-3.47077199058619E-08"
-        izz="0.000833137426033134" />
+        xyz="2.9549E-17 -0.00030197 0.11134"
+        rpy="0 0 0" />
+      <mass
+        value="17.843" />
+      <inertia
+        ixx="0.87104"
+        ixy="-3.2142E-07"
+        ixz="-9.442E-18"
+        iyy="0.48766"
+        iyz="0.00055476"
+        izz="0.98951" />
     </inertial>
     <visual>
@@ -50,5 +75,5 @@
         name="">
         <color
-          rgba="0.792156862745098 0.819607843137255 0.933333333333333 1" />
+          rgba="0.41569 0.67451 1 1" />
       </material>
     </visual>
@@ -63,4 +88,5 @@
     </collision>
   </link>
+  <!-- World Joint For Fixed Base -->
   <joint name="fixed_base" type="fixed">
     <parent link="world" />
@@ -68,18 +94,124 @@
   </joint>
   <link
+    name="camera_link">
+    <inertial>
+      <origin
+        xyz="-3.8492E-19 0.0043066 -0.0086877"
+        rpy="0 0 0" />
+      <mass
+        value="0.011" />
+      <inertia
+        ixx="1.206E-06"
+        ixy="1.0009E-22"
+        ixz="-5.0667E-23"
+        iyy="1.4269E-06"
+        iyz="8.5819E-08"
+        izz="1.3248E-06" />
+    </inertial>
+    <visual>
+      <origin
+        xyz="0 0 0"
+        rpy="0 0 0" />
+      <geometry>
+        <mesh
+          filename="package://project_two/meshes/camera_link.STL" />
+      </geometry>
+      <material
+        name="">
+        <color
+          rgba="0.19608 0.19608 0.19608 1" />
+      </material>
+    </visual>
+    <collision>
+      <origin
+        xyz="0 0 0"
+        rpy="0 0 0" />
+      <geometry>
+        <mesh
+          filename="package://project_two/meshes/camera_link.STL" />
+      </geometry>
+    </collision>
+  </link>
+  <joint
+    name="camera_joint"
+    type="fixed">
+    <origin
+      xyz="0 -0.120050000000001 0.2983"
+      rpy="1.5707963267949 0 0" />
+    <parent
+      link="base_link" />
+    <child
+      link="camera_link" />
+    <axis
+      xyz="0 0 0" />
+  </joint>
+  <link
+    name="link_0">
+    <inertial>
+      <origin
+        xyz="0.00081893 -0.00081893 0.50768"
+        rpy="0 0 0" />
+      <mass
+        value="0.36506" />
+      <inertia
+        ixx="0.00051381"
+        ixy="-1.2538E-05"
+        ixz="3.4706E-08"
+        iyy="0.00051381"
+        iyz="-3.4708E-08"
+        izz="0.00083314" />
+    </inertial>
+    <visual>
+      <origin
+        xyz="0 0 0"
+        rpy="0 0 0" />
+      <geometry>
+        <mesh
+          filename="package://project_two/meshes/link_0.STL" />
+      </geometry>
+      <material
+        name="">
+        <color
+          rgba="0.79216 0.81961 0.93333 1" />
+      </material>
+    </visual>
+    <collision>
+      <origin
+        xyz="0 0 0"
+        rpy="0 0 0" />
+      <geometry>
+        <mesh
+          filename="package://project_two/meshes/link_0.STL" />
+      </geometry>
+    </collision>
+  </link>
+  <joint
+    name="joint_0"
+    type="fixed">
+    <origin
+      xyz="0 0 0"
+      rpy="0 0 0" />
+    <parent
+      link="base_link" />
+    <child
+      link="link_0" />
+    <axis
+      xyz="0 0 0" />
+  </joint>
+  <link
     name="link_1">
     <inertial>
       <origin
-        xyz="-2.01994143885152E-08 0.0147276350283187 0.0810226747554533"
-        rpy="0 0 0" />
-      <mass
-        value="1.21747724894722" />
-      <inertia
-        ixx="0.00255263718574973"
-        ixy="7.20416731900228E-09"
-        ixz="-3.70618686006579E-09"
-        iyy="0.00210897804842468"
-        iyz="-0.000297852263493"
-        izz="0.00266305849374601" />
+        xyz="-1.7916E-08 0.014728 0.57467"
+        rpy="0 0 0" />
+      <mass
+        value="1.2175" />
+      <inertia
+        ixx="0.0025526"
+        ixy="5.0045E-09"
+        ixz="5.1533E-10"
+        iyy="0.002109"
+        iyz="-0.00029785"
+        izz="0.0026631" />
     </inertial>
     <visual>
@@ -94,5 +226,5 @@
         name="">
         <color
-          rgba="0.796078431372549 0.819607843137255 0.933333333333333 1" />
+          rgba="0.79608 0.81961 0.93333 1" />
       </material>
     </visual>
@@ -114,5 +246,5 @@
       rpy="0 0 0" />
     <parent
-      link="base_link" />
+      link="link_0" />
     <child
       link="link_1" />
@@ -124,5 +256,6 @@
       effort="0"
       velocity="0" />
-    <dynamics damping="0.7" friction="1.0"/>
+      <!-- Added Joint Dynamics to Prevent Separation -->
+      <dynamics damping="0.7" friction="1.0"/>
   </joint>
   <link
@@ -130,15 +263,15 @@
     <inertial>
       <origin
-        xyz="1.42302771372066E-07 -0.00806677437392857 0.138671119640996"
-        rpy="0 0 0" />
-      <mass
-        value="0.330021171721498" />
-      <inertia
-        ixx="0.000313864807069818"
-        ixy="1.39841178897165E-09"
-        ixz="2.28303347219796E-10"
-        iyy="0.000335340499862343"
-        iyz="-7.39635181857418E-05"
-        izz="0.000541751266552296" />
+        xyz="1.423E-07 -0.0080668 0.63232"
+        rpy="0 0 0" />
+      <mass
+        value="0.33002" />
+      <inertia
+        ixx="0.00031386"
+        ixy="1.3984E-09"
+        ixz="2.283E-10"
+        iyy="0.00033534"
+        iyz="-7.3964E-05"
+        izz="0.00054175" />
     </inertial>
     <visual>
@@ -153,5 +286,5 @@
         name="">
         <color
-          rgba="0.482352941176471 0.792156862745098 1 1" />
+          rgba="0.48235 0.79216 1 1" />
       </material>
     </visual>
@@ -166,10 +299,21 @@
     </collision>
   </link>
-  <joint name="link_1_cap_joint" type="prismatic">
-      <origin xyz="0 0 0" rpy="0 0 0" />
-      <parent link="link_1" />
-      <child link="link_1_cap" />
-      <axis xyz="1 0 0" />
-      <limit lower="0" upper="0" effort="0" velocity="0" />
+  <joint
+    name="link_1_cap_joint"
+    type="prismatic">
+    <origin
+      xyz="0 0 0"
+      rpy="0 0 0" />
+    <parent
+      link="link_1" />
+    <child
+      link="link_1_cap" />
+    <axis
+      xyz="0 0 1" />
+    <limit
+      lower="0"
+      upper="0"
+      effort="0"
+      velocity="0" />
   </joint>
   <link
@@ -177,15 +321,15 @@
     <inertial>
       <origin
-        xyz="5.28224377692258E-09 -0.212110309879065 0.129614412124911"
-        rpy="0 0 0" />
-      <mass
-        value="4.0347772255313" />
-      <inertia
-        ixx="0.112004707514996"
-        ixy="1.49514812132019E-08"
-        ixz="-4.44365415979749E-10"
-        iyy="0.00580966202350412"
-        iyz="1.87193857431351E-05"
-        izz="0.1121524014166" />
+        xyz="5.2822E-09 -0.21211 0.12961"
+        rpy="0 0 0" />
+      <mass
+        value="4.0348" />
+      <inertia
+        ixx="0.112"
+        ixy="1.4951E-08"
+        ixz="-4.4437E-10"
+        iyy="0.0058097"
+        iyz="1.8719E-05"
+        izz="0.11215" />
     </inertial>
     <visual>
@@ -200,5 +344,5 @@
         name="">
         <color
-          rgba="0.792156862745098 0.819607843137255 0.933333333333333 1" />
+          rgba="0.79216 0.81961 0.93333 1" />
       </material>
     </visual>
@@ -217,6 +361,6 @@
     type="revolute">
     <origin
-      xyz="0 0 0.09"
-      rpy="-1.5707963267949 0 0" />
+      xyz="0 0 0.58365"
+      rpy="-1.57079632679489 0 0" />
     <parent
       link="link_1" />
@@ -230,5 +374,6 @@
       effort="0"
       velocity="0" />
-    <dynamics damping="0.7" friction="1.0"/>
+      <!-- Added Joint Dynamics to Prevent Separation -->
+      <dynamics damping="0.7" friction="1.0"/>
   </joint>
   <link
@@ -236,15 +381,15 @@
     <inertial>
       <origin
-        xyz="-1.42302772727024E-07 0.00806677437392862 0.183671119640996"
-        rpy="0 0 0" />
-      <mass
-        value="0.330021171721499" />
-      <inertia
-        ixx="0.000313864807069819"
-        ixy="1.39841178841114E-09"
-        ixz="-2.28303348779531E-10"
-        iyy="0.000335340499862345"
-        iyz="7.39635181857419E-05"
-        izz="0.000541751266552297" />
+        xyz="-1.423E-07 0.0080668 0.18367"
+        rpy="0 0 0" />
+      <mass
+        value="0.33002" />
+      <inertia
+        ixx="0.00031386"
+        ixy="1.3984E-09"
+        ixz="-2.283E-10"
+        iyy="0.00033534"
+        iyz="7.3964E-05"
+        izz="0.00054175" />
     </inertial>
     <visual>
@@ -259,5 +404,5 @@
         name="">
         <color
-          rgba="0.482352941176471 0.792156862745098 1 1" />
+          rgba="0.48235 0.79216 1 1" />
       </material>
     </visual>
@@ -272,10 +417,21 @@
     </collision>
   </link>
-  <joint name="link_2_cap_1_joint" type="prismatic">
-      <origin xyz="0 0 0" rpy="0 0 0" />
-      <parent link="link_2" />
-      <child link="link_2_cap_1" />
-      <axis xyz="1 0 0" />
-      <limit lower="0" upper="0" effort="0" velocity="0" />
+  <joint
+    name="link_2_cap_1_joint"
+    type="prismatic">
+    <origin
+      xyz="0 0 0"
+      rpy="0 0 0" />
+    <parent
+      link="link_2" />
+    <child
+      link="link_2_cap_1" />
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
Commit message: dummy controller added, all elements spawning in rviz successfully

File: project_two/urdf/robot_arm.urdf.xacro (robot description, xacro)
@@ -1,6 +1,3 @@
 <?xml version="1.0" ?>
-<!-- This URDF was automatically created by SolidWorks to URDF Exporter! Originally created by Stephen Brawner (brawner@gmail.com)
-     Commit Version: 1.6.0-4-g7f85cfe  Build Version: 1.6.7995.38578
-     For more information, please see http://wiki.ros.org/sw_urdf_exporter -->
 <robot
   name="robot_arm" xmlns:xacro="http://ros.org/wiki/xacro">
@@ -1061,4 +1058,41 @@
         <state_interface name="position"/>
     </joint>
+    <!-- Dummy Controller for Link Cap joints to instantiate in Rviz -->
+    <joint name="link_1_cap_joint">
+        <command_interface name="position"/>
+        <state_interface name="position"/>
+    </joint>
+    <joint name="link_2_cap_joint">
+        <command_interface name="position"/>
+        <state_interface name="position"/>
+    </joint>
+    <joint name="link_3_cap_joint">
+        <command_interface name="position"/>
+        <state_interface name="position"/>
+    </joint>
+    <joint name="link_4_cap_joint">
+        <command_interface name="position"/>
+        <state_interface name="position"/>
+    </joint>
+    <joint name="link_5_cap_joint">
+        <command_interface name="position"/>
+        <state_interface name="position"/>
+    </joint>
+    <joint name="link_6_cap_joint">
+        <command_interface name="position"/>
+        <state_interface name="position"/>
+    </joint>
+    <joint name="tooling_joint">
+        <command_interface name="position"/>
+        <state_interface name="position"/>
+    </joint>
+    <joint name="link_2_cap_2_joint">
+        <command_interface name="position"/>
+        <state_interface name="position"/>
+    </joint>
+    <joint name="link_2_cap_1_joint">
+        <command_interface name="position"/>
+        <state_interface name="position"/>
+    </joint>
   </ros2_control>
   <!-- Control Configuration File -->

Commit message: camera plugin added but not publishing

File: project_two/urdf/robot_arm.urdf.xacro (robot description, xacro)
@@ -90,4 +90,17 @@
     <child link="base_link" />
   </joint>
+  <joint
+    name="camera_joint"
+    type="fixed">
+    <origin
+      xyz="0 -0.120050000000001 0.2983"
+      rpy="1.5707963267949 0 0" />
+    <parent
+      link="base_link" />
+    <child
+      link="camera_link" />
+    <axis
+      xyz="0 0 0" />
+  </joint>
   <link
     name="camera_link">
@@ -130,17 +143,11 @@
     </collision>
   </link>
-  <joint
-    name="camera_joint"
-    type="fixed">
-    <origin
-      xyz="0 -0.120050000000001 0.2983"
-      rpy="1.5707963267949 0 0" />
-    <parent
-      link="base_link" />
-    <child
-      link="camera_link" />
-    <axis
-      xyz="0 0 0" />
-  </joint>
+  <!-- Dummy link to correct Image Reference Frame for Camera -->
+  <joint name="camera_optical_joint" type="fixed">
+      <origin xyz="0 0 0" rpy="0 -1.5707 -1.5707963267949" />
+      <parent link="camera_link" />
+      <child link="camera_link_optical" />
+  </joint>
+  <link name="camera_link_optical"></link>
   <link
     name="link_0">
@@ -1063,8 +1070,4 @@
         <state_interface name="position"/>
     </joint>
-    <joint name="link_2_cap_joint">
-        <command_interface name="position"/>
-        <state_interface name="position"/>
-    </joint>
     <joint name="link_3_cap_joint">
         <command_interface name="position"/>
@@ -1076,8 +1079,4 @@
     </joint>
     <joint name="link_5_cap_joint">
-        <command_interface name="position"/>
-        <state_interface name="position"/>
-    </joint>
-    <joint name="link_6_cap_joint">
         <command_interface name="position"/>
         <state_interface name="position"/>
@@ -1121,3 +1120,30 @@
     <implicitSpringDamper>true</implicitSpringDamper>
   </gazebo>
+  <!-- Camera Sensor -->
+  <gazebo reference="camera_link_optical">
+    <sensor name="camera_sensor" type="camera">
+      <pose> 0 0 0 0 0 0</pose>
+      <visualize>true</visualize>
+      <update_rate>10</update_rate>
+      <camera>
+        <horizontal_fov>1.089</horizontal_fov>
+        <image>
+            <format>R8G8B8</format>
+            <width>640</width>
+            <height>480</height>
+        </image>
+        <clip>
+            <near>0.05</near>
+            <far>20</far>
+        </clip>
+      </camera>
+      <plugin name="camera_controller" filename="libgazebo_ros_camera.so">
+        <always_on>true</always_on>
+        <cameraName>camera</cameraName>
+        <imageTopicName>image_raw</imageTopicName>
+        <cameraInfoTopicName>camera_info</cameraInfoTopicName>
+        <frame_name>camera_link_optical</frame_name>
+      </plugin>
+    </sensor>
+  </gazebo>
 </robot>

Commit message: Fixed Camera Topic Issues

File: project_two/urdf/robot_arm.urdf.xacro (robot description, xacro)
@@ -144,4 +144,5 @@
   </link>
   <!-- Dummy link to correct Image Reference Frame for Camera -->
+  <link name="camera_link_optical" />
   <joint name="camera_optical_joint" type="fixed">
       <origin xyz="0 0 0" rpy="0 -1.5707 -1.5707963267949" />
@@ -149,5 +150,4 @@
       <child link="camera_link_optical" />
   </joint>
-  <link name="camera_link_optical"></link>
   <link
     name="link_0">
@@ -1122,5 +1122,5 @@
   <!-- Camera Sensor -->
   <gazebo reference="camera_link_optical">
-    <sensor name="camera_sensor" type="camera">
+    <sensor name="camera" type="camera">
       <pose> 0 0 0 0 0 0</pose>
       <visualize>true</visualize>
