Commit message: controller added, spawns without controller but not with

File: humanoid/urdf/humanoid.urdf.xacro (robot description, xacro)
@@ -1,8 +1,6 @@
-<?xml version="1.0" encoding="utf-8"?>
-<!-- This URDF was automatically created by SolidWorks to URDF Exporter! Originally created by Stephen Brawner (brawner@gmail.com)
-     Commit Version: 1.6.0-4-g7f85cfe  Build Version: 1.6.7995.38578
-     For more information, please see http://wiki.ros.org/sw_urdf_exporter -->
+<?xml version="1.0" ?>
 <robot
   name="humanoid" xmlns:xacro="http://ros.org/wiki/xacro">
+  <link name="dummy_link"></link>
   <link
     name="base_link">
@@ -45,4 +43,9 @@
     </collision>
   </link>
+  <joint name="dummy_joint" type="fixed">
+    <origin rpy="0 0 0" xyz="0 0 0" />
+    <parent link="dummy_link"/>
+    <child link="base_link"/>
+  </joint>
   <link
     name="hd_link">
@@ -487,5 +490,5 @@
   </link>
   <joint
-    name="l_shldr_2_joint"
+    name="l_shldr_1_joint"
     type="revolute">
     <origin
@@ -1548,3 +1551,190 @@
       velocity="0" />
   </joint>
+  <!-- Start of Controllers -->
+  <ros2_control name="GazeboSystem" type="system">
+    <hardware>
+      <plugin>gazebo_ros2_control/GazeboSystem</plugin>
+    </hardware>
+    <!-- Position Controller -->
+    <joint name="hd_joint">
+      <command_interface name="position">
+        <param name="min">-1.5708</param>
+        <param name="max">1.5708</param>
+      </command_interface>
+      <state_interface name="position"/>
+    </joint>
+    <joint name="r_shldr_1_joint">
+      <command_interface name="position">
+        <param name="min">-1.5708</param>
+        <param name="max">1.5708</param>
+      </command_interface>
+      <state_interface name="position"/>
+    </joint>
+    <joint name="r_shldr_2_joint">
+      <command_interface name="position">
+        <param name="min">-1.5708</param>
+        <param name="max">1.5708</param>
+      </command_interface>
+      <state_interface name="position"/>
+    </joint>
+    <joint name="r_elb_1_joint">
+      <command_interface name="position">
+        <param name="min">-1.5708</param>
+        <param name="max">1.5708</param>
+      </command_interface>
+      <state_interface name="position"/>
+    </joint>
+    <joint name="r_elb_2_joint">
+      <command_interface name="position">
+        <param name="min">-1.5708</param>
+        <param name="max">1.5708</param>
+      </command_interface>
+      <state_interface name="position"/>
+    </joint>
+    <joint name="r_wst_joint">
+      <command_interface name="position">
+        <param name="min">-3.1416</param>
+        <param name="max">3.1416</param>
+      </command_interface>
+      <state_interface name="position"/>
+    </joint>
+    <joint name="l_shldr_1_joint">
+      <command_interface name="position">
+        <param name="min">-1.5708</param>
+        <param name="max">1.5708</param>
+      </command_interface>
+      <state_interface name="position"/>
+    </joint>
+    <joint name="l_shldr_2_joint">
+      <command_interface name="position">
+        <param name="min">-1.5708</param>
+        <param name="max">1.5708</param>
+      </command_interface>
+      <state_interface name="position"/>
+    </joint>
+    <joint name="l_elb_1_joint">
+      <command_interface name="position">
+        <param name="min">-1.5708</param>
+        <param name="max">1.5708</param>
+      </command_interface>
+      <state_interface name="position"/>
+    </joint>
+    <joint name="l_elb_2_joint">
+      <command_interface name="position">
+        <param name="min">-1.5708</param>
+        <param name="max">1.5708</param>
+      </command_interface>
+      <state_interface name="position"/>
+    </joint>
+    <joint name="l_wst_joint">
+      <command_interface name="position">
+        <param name="min">-3.1416</param>
+        <param name="max">3.1416</param>
+      </command_interface>
+      <state_interface name="position"/>
+    </joint>
+    <joint name="r_hp_1_joint">
+      <command_interface name="position">
+        <param name="min">-1.5708</param>
+        <param name="max">1.5708</param>
+      </command_interface>
+      <state_interface name="position"/>
+    </joint>
+    <joint name="r_hp_2_joint">
+      <command_interface name="position">
+        <param name="min">-1.5708</param>
+        <param name="max">1.5708</param>
+      </command_interface>
+      <state_interface name="position"/>
+    </joint>
+    <joint name="r_kn_joint">
+      <command_interface name="position">
+        <param name="min">0</param>
+        <param name="max">1.5708</param>
+      </command_interface>
+      <state_interface name="position"/>
+    </joint>
+    <joint name="r_ank_1_joint">
+      <command_interface name="position">
+        <param name="min">-1.5708</param>
+        <param name="max">1.5708</param>
+      </command_interface>
+      <state_interface name="position"/>
+    </joint>
+    <joint name="r_ank_2_joint">
+      <command_interface name="position">
+        <param name="min">-0.7854</param>
+        <param name="max">0.7854</param>
+      </command_interface>
+      <state_interface name="position"/>
+    </joint>
+    <joint name="r_str_joint">
+      <command_interface name="position">
+        <param name="min">-3.1416</param>
+        <param name="max">3.1416</param>
+      </command_interface>
+      <state_interface name="position"/>
+    </joint>
+    <joint name="r_wl_joint">
+      <command_interface name="position">
+        <param name="min">-3.1416</param>
+        <param name="max">3.1416</param>
+      </command_interface>
+      <state_interface name="position"/>
+    </joint>
+    <joint name="l_hp_1_joint">
+      <command_interface name="position">
+        <param name="min">-1.5708</param>
+        <param name="max">1.5708</param>
+      </command_interface>
+      <state_interface name="position"/>
+    </joint>
+    <joint name="l_hp_2_joint">
+      <command_interface name="position">
+        <param name="min">-1.5708</param>
+        <param name="max">1.5708</param>
+      </command_interface>
+      <state_interface name="position"/>
+    </joint>
+    <joint name="l_kn_joint">
+      <command_interface name="position">
+        <param name="min">0</param>
+        <param name="max">1.5708</param>
+      </command_interface>
+      <state_interface name="position"/>
+    </joint>
+    <joint name="l_ank_1_joint">
+      <command_interface name="position">
+        <param name="min">-1.5708</param>
+        <param name="max">1.5708</param>
+      </command_interface>
+      <state_interface name="position"/>
+    </joint>
+    <joint name="l_ank_2_joint">
+      <command_interface name="position">
+        <param name="min">-0.7854</param>
+        <param name="max">0.7854</param>
+      </command_interface>
+      <state_interface name="position"/>
+    </joint>
+    <joint name="l_str_joint">
+      <command_interface name="position">
+        <param name="min">-3.1416</param>
+        <param name="max">3.1416</param>
+      </command_interface>
+      <state_interface name="position"/>
+    </joint>
+    <joint name="l_wl_joint">
+      <command_interface name="position">
+        <param name="min">-3.1416</param>
+        <param name="max">3.1416</param>
+      </command_interface>
+      <state_interface name="position"/>
+    </joint>
+  </ros2_control>
+  <gazebo>
+    <plugin filename="libgazebo_ros2_control.so" name="gazebo_ros2_control">
+      <parameters>$(find humanoid)/config/control.yaml</parameters>
+    </plugin>
+  </gazebo>
 </robot>

Commit message: Resolved Visualization Issues

File: humanoid/urdf/humanoid.urdf.xacro (robot description, xacro)
@@ -2,4 +2,5 @@
 <robot
   name="humanoid" xmlns:xacro="http://ros.org/wiki/xacro">
+  <!-- Dummy Link -->
   <link name="dummy_link"></link>
   <link
@@ -43,4 +44,5 @@
     </collision>
   </link>
+  <!-- Dummy Joint -->
   <joint name="dummy_joint" type="fixed">
     <origin rpy="0 0 0" xyz="0 0 0" />
@@ -1551,186 +1553,186 @@
       velocity="0" />
   </joint>
-  <!-- Start of Controllers -->
+  <!-- Controller Plugin -->
   <ros2_control name="GazeboSystem" type="system">
     <hardware>
-      <plugin>gazebo_ros2_control/GazeboSystem</plugin>
+        <plugin>gazebo_ros2_control/GazeboSystem</plugin>
     </hardware>
     <!-- Position Controller -->
     <joint name="hd_joint">
-      <command_interface name="position">
-        <param name="min">-1.5708</param>
-        <param name="max">1.5708</param>
-      </command_interface>
-      <state_interface name="position"/>
+        <command_interface name="position">
+            <param name="min">-1.5708</param>
+            <param name="max">1.5708</param>
+        </command_interface>
+        <state_interface name="position"/>
     </joint>
     <joint name="r_shldr_1_joint">
-      <command_interface name="position">
-        <param name="min">-1.5708</param>
-        <param name="max">1.5708</param>
-      </command_interface>
-      <state_interface name="position"/>
+        <command_interface name="position">
+            <param name="min">-1.5708</param>
+            <param name="max">1.5708</param>
+        </command_interface>
+        <state_interface name="position"/>
     </joint>
     <joint name="r_shldr_2_joint">
-      <command_interface name="position">
-        <param name="min">-1.5708</param>
-        <param name="max">1.5708</param>
-      </command_interface>
-      <state_interface name="position"/>
+        <command_interface name="position">
+            <param name="min">-1.5708</param>
+            <param name="max">1.5708</param>
+        </command_interface>
+        <state_interface name="position"/>
     </joint>
     <joint name="r_elb_1_joint">
-      <command_interface name="position">
-        <param name="min">-1.5708</param>
-        <param name="max">1.5708</param>
-      </command_interface>
-      <state_interface name="position"/>
+        <command_interface name="position">
+            <param name="min">-1.5708</param>
+            <param name="max">1.5708</param>
+        </command_interface>
+        <state_interface name="position"/>
     </joint>
     <joint name="r_elb_2_joint">
-      <command_interface name="position">
-        <param name="min">-1.5708</param>
-        <param name="max">1.5708</param>
-      </command_interface>
-      <state_interface name="position"/>
+        <command_interface name="position">
+            <param name="min">-1.5708</param>
+            <param name="max">1.5708</param>
+        </command_interface>
+        <state_interface name="position"/>
     </joint>
     <joint name="r_wst_joint">
-      <command_interface name="position">
-        <param name="min">-3.1416</param>
-        <param name="max">3.1416</param>
-      </command_interface>
-      <state_interface name="position"/>
+        <command_interface name="position">
+            <param name="min">-3.1416</param>
+            <param name="max">3.1416</param>
+        </command_interface>
+        <state_interface name="position"/>
     </joint>
     <joint name="l_shldr_1_joint">
-      <command_interface name="position">
-        <param name="min">-1.5708</param>
-        <param name="max">1.5708</param>
-      </command_interface>
-      <state_interface name="position"/>
+        <command_interface name="position">
+            <param name="min">-1.5708</param>
+            <param name="max">1.5708</param>
+        </command_interface>
+        <state_interface name="position"/>
     </joint>
     <joint name="l_shldr_2_joint">
-      <command_interface name="position">
-        <param name="min">-1.5708</param>
-        <param name="max">1.5708</param>
-      </command_interface>
-      <state_interface name="position"/>
+        <command_interface name="position">
+            <param name="min">-1.5708</param>
+            <param name="max">1.5708</param>
+        </command_interface>
+        <state_interface name="position"/>
     </joint>
     <joint name="l_elb_1_joint">
-      <command_interface name="position">
-        <param name="min">-1.5708</param>
-        <param name="max">1.5708</param>
-      </command_interface>
-      <state_interface name="position"/>
+        <command_interface name="position">
+            <param name="min">-1.5708</param>
+            <param name="max">1.5708</param>
+        </command_interface>
+        <state_interface name="position"/>
     </joint>
     <joint name="l_elb_2_joint">
-      <command_interface name="position">
-        <param name="min">-1.5708</param>
-        <param name="max">1.5708</param>
-      </command_interface>
-      <state_interface name="position"/>
+        <command_interface name="position">
+            <param name="min">-1.5708</param>
+            <param name="max">1.5708</param>
+        </command_interface>
+        <state_interface name="position"/>
     </joint>
     <joint name="l_wst_joint">
-      <command_interface name="position">
-        <param name="min">-3.1416</param>
-        <param name="max">3.1416</param>
-      </command_interface>
-      <state_interface name="position"/>
+        <command_interface name="position">
+            <param name="min">-3.1416</param>
+            <param name="max">3.1416</param>
+        </command_interface>
+        <state_interface name="position"/>
     </joint>
     <joint name="r_hp_1_joint">
-      <command_interface name="position">
-        <param name="min">-1.5708</param>
-        <param name="max">1.5708</param>
-      </command_interface>
-      <state_interface name="position"/>
+        <command_interface name="position">
+            <param name="min">-1.5708</param>
+            <param name="max">1.5708</param>
+        </command_interface>
+        <state_interface name="position"/>
     </joint>
     <joint name="r_hp_2_joint">
-      <command_interface name="position">
-        <param name="min">-1.5708</param>
-        <param name="max">1.5708</param>
-      </command_interface>
-      <state_interface name="position"/>
+        <command_interface name="position">
+            <param name="min">-1.5708</param>
+            <param name="max">1.5708</param>
+        </command_interface>
+        <state_interface name="position"/>
     </joint>
     <joint name="r_kn_joint">
-      <command_interface name="position">
-        <param name="min">0</param>
-        <param name="max">1.5708</param>
-      </command_interface>
-      <state_interface name="position"/>
+        <command_interface name="position">
+            <param name="min">0.0</param>
+            <param name="max">1.5708</param>
+        </command_interface>
+        <state_interface name="position"/>
     </joint>
     <joint name="r_ank_1_joint">
-      <command_interface name="position">
-        <param name="min">-1.5708</param>
-        <param name="max">1.5708</param>
-      </command_interface>
-      <state_interface name="position"/>
+        <command_interface name="position">
+            <param name="min">-1.5708</param>
+            <param name="max">1.5708</param>
+        </command_interface>
+        <state_interface name="position"/>
     </joint>
     <joint name="r_ank_2_joint">
-      <command_interface name="position">
-        <param name="min">-0.7854</param>
-        <param name="max">0.7854</param>
-      </command_interface>
-      <state_interface name="position"/>
+        <command_interface name="position">
+            <param name="min">-0.7854</param>
+            <param name="max">0.7854</param>
+        </command_interface>
+        <state_interface name="position"/>
     </joint>
     <joint name="r_str_joint">
-      <command_interface name="position">
-        <param name="min">-3.1416</param>
-        <param name="max">3.1416</param>
-      </command_interface>
-      <state_interface name="position"/>
+        <command_interface name="position">
+            <param name="min">-3.1416</param>
+            <param name="max">3.1416</param>
+        </command_interface>
+        <state_interface name="position"/>
     </joint>
     <joint name="r_wl_joint">
-      <command_interface name="position">
-        <param name="min">-3.1416</param>
-        <param name="max">3.1416</param>
-      </command_interface>
-      <state_interface name="position"/>
+        <command_interface name="position">
+            <param name="min">-3.1416</param>
+            <param name="max">3.1416</param>
+        </command_interface>
+        <state_interface name="position"/>
     </joint>
     <joint name="l_hp_1_joint">
-      <command_interface name="position">
-        <param name="min">-1.5708</param>
-        <param name="max">1.5708</param>
-      </command_interface>
-      <state_interface name="position"/>
+        <command_interface name="position">
+            <param name="min">-1.5708</param>
+            <param name="max">1.5708</param>
+        </command_interface>
+        <state_interface name="position"/>
     </joint>
     <joint name="l_hp_2_joint">
-      <command_interface name="position">
-        <param name="min">-1.5708</param>
-        <param name="max">1.5708</param>
-      </command_interface>
-      <state_interface name="position"/>
+        <command_interface name="position">
+            <param name="min">-1.5708</param>
+            <param name="max">1.5708</param>
+        </command_interface>
+        <state_interface name="position"/>
     </joint>
     <joint name="l_kn_joint">
-      <command_interface name="position">
-        <param name="min">0</param>
-        <param name="max">1.5708</param>
-      </command_interface>
-      <state_interface name="position"/>
+        <command_interface name="position">
+            <param name="min">0.0</param>
+            <param name="max">1.5708</param>
+        </command_interface>
+        <state_interface name="position"/>
     </joint>
     <joint name="l_ank_1_joint">
-      <command_interface name="position">
-        <param name="min">-1.5708</param>
-        <param name="max">1.5708</param>
-      </command_interface>
-      <state_interface name="position"/>
+        <command_interface name="position">
+            <param name="min">-1.5708</param>
+            <param name="max">1.5708</param>
+        </command_interface>
+        <state_interface name="position"/>
     </joint>
     <joint name="l_ank_2_joint">
-      <command_interface name="position">
-        <param name="min">-0.7854</param>
-        <param name="max">0.7854</param>
-      </command_interface>
-      <state_interface name="position"/>
+        <command_interface name="position">
+            <param name="min">-0.7854</param>
+            <param name="max">0.7854</param>
+        </command_interface>
+        <state_interface name="position"/>
     </joint>
     <joint name="l_str_joint">
-      <command_interface name="position">
-        <param name="min">-3.1416</param>
-        <param name="max">3.1416</param>
-      </command_interface>
-      <state_interface name="position"/>
+        <command_interface name="position">
+            <param name="min">-3.1416</param>
+            <param name="max">3.1416</param>
+        </command_interface>
+        <state_interface name="position"/>
     </joint>
     <joint name="l_wl_joint">
-      <command_interface name="position">
-        <param name="min">-3.1416</param>
-        <param name="max">3.1416</param>
-      </command_interface>
-      <state_interface name="position"/>
-    </joint>
-  </ros2_control>
+        <command_interface name="position">
+            <param name="min">-3.1416</param>
+            <param name="max">3.1416</param>
+        </command_interface>
+        <state_interface name="position"/>
+    </joint>
+ </ros2_control>
   <gazebo>
     <plugin filename="libgazebo_ros2_control.so" name="gazebo_ros2_control">
@@ -1738,46 +1740,39 @@
     </plugin>
   </gazebo>
+  <!-- LiDAR Plugin -->
   <gazebo reference="ldr_link">
-    <sensor name="lidar" type="ray">
-      <pose>0.0 0.0 0.0 0 0 0</pose>
-      <always_on>true</always_on>
-      <visualize>true</visualize>
-      <update_rate>5</update_rate>
-      <ray>
-        <scan>
-          <horizontal>
-            <samples>360</samples>
-            <resolution>1.00000</resolution>
-            <min_angle>0.000000</min_angle>
-            <max_angle>6.280000</max_angle>
-          </horizontal>
-        </scan>
-        <range>
-          <min>0.120000</min>
-          <max>3.5</max>
-          <resolution>0.015000</resolution>
-        </range>
-        <noise>
-          <type>gaussian</type>
-          <mean>0.0</mean>
-          <stddev>0.01</stddev>
-        </noise>
-      </ray>
-      <plugin name="scan" filename="libgazebo_ros_ray_sensor.so">
-        <ros>
-          <remapping>~/out:=scan</remapping>
-        </ros>
-        <output_type>sensor_msgs/LaserScan</output_type>
-        <frame_name>ldr_link</frame_name>
-      </plugin>
-    </sensor>
-  </gazebo>
-  <gazebo>
-    <plugin filename="libodometry_plugin.so" name="odometry_plugin">
-      <!-- Name of the link for which the odometry is required -->
-      <frame>dummy_link</frame>
-      <!-- Any arbitray name for the world frame -->
-      <world_frame>fixed_world</world_frame>
+  <sensor name="lidar" type="ray">
+    <pose>0.0 0.0 0.0 0 0 0</pose>
+    <always_on>true</always_on>
+    <visualize>true</visualize>
+    <update_rate>5</update_rate>
+    <ray>
+      <scan>
+        <horizontal>
+          <samples>360</samples>
+          <resolution>1.00000</resolution>
+          <min_angle>0.000000</min_angle>
+          <max_angle>6.280000</max_angle>
+        </horizontal>
+      </scan>
+      <range>
+        <min>0.120000</min>
+        <max>3.5</max>
+        <resolution>0.015000</resolution>
+      </range>
+      <noise>
+        <type>gaussian</type>
+        <mean>0.0</mean>
+        <stddev>0.01</stddev>
+      </noise>
+    </ray>
+    <plugin name="scan" filename="libgazebo_ros_ray_sensor.so">
+      <ros>
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